File: canProtoshieldArduinoMega/canprotoshield.brd (EAGLE design)
At the start: 100 x 80 mm, 55 parts, among them CN1 1X4-3.5MM, CN10 1X4-3.5MM, CN11 1X4-3.5MM, CN12 1X4-3.5MM, CN13 1X4-3.5MM, CN14 1X4-3.5MM, CN15 1X4-3.5MM, CN16 1X4-3.5MM, CN17 1X4-3.5MM, CN18 1X4-3.5MM, CN19 1X4-3.5MM, CN2 1X4-3.5MM, CN20 1X4-3.5MM, CN21 1X4-3.5MM, CN22 1X4-3.5MM, CN23 1X4-3.5MM, CN24 1X4-3.5MM, CN25 1X4-3.5MM, CN26 1X4-3.5MM, CN27 1X4-3.5MM, CN28 1X4-3.5MM, CN29 1X4-3.5MM, CN3 1X4-3.5MM, CN30 1X4-3.5MM, CN31 1X4-3.5MM, CN32 1X4-3.5MM, CN33 1X4-3.5MM, CN34 1X4-3.5MM, CN4 1X4-3.5MM, CN5 1X4-3.5MM, CN6 1X4-3.5MM, CN7 1X4-3.5MM, CN8 1X4-3.5MM, CN9 1X4-3.5MM, U2 MCP2551, U3 ARDUINO-MEGAFULL

Commit message: Wiring.
Connections:
- removed net N$31: BUS_GND.1
- net GND: now also BUS_GND.1
Routing:
- net VCC: track 0.00 -> 234.0 mm, vias 0 -> 2
- net GND: track 0.00 -> 224.3 mm
- net MCP_SCK: track 0.00 -> 97.9 mm
- net MCP_CS: track 0.00 -> 92.1 mm
- net 22: track 6.88 -> 97.0 mm, vias 0 -> 1
- net MCP_SI: track 0.00 -> 88.6 mm, vias 0 -> 3
- net MCP_SO: track 0.00 -> 84.6 mm, vias 0 -> 1
- net 47: track 0.00 -> 29.3 mm
- net A0: track 0.00 -> 27.7 mm
- net 46: track 0.00 -> 26.6 mm
- net A1: track 0.00 -> 25.4 mm
- net A2: track 0.00 -> 24.5 mm
- net 45: track 0.00 -> 23.8 mm, vias 0 -> 1
- net A3: track 0.00 -> 23.5 mm
- net N$9: track 0.00 -> 23.4 mm
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