File: canProtoshieldArduinoMega/canprotoshield_eth.brd (EAGLE design)
At the start: 101.3 x 80.6 mm, 58 parts, among them CN1 1X4-3.5MM, CN10 1X4-3.5MM, CN11 1X4-3.5MM, CN12 1X4-3.5MM, CN13 1X4-3.5MM, CN14 1X4-3.5MM, CN15 1X4-3.5MM, CN16 1X4-3.5MM, CN17 1X4-3.5MM, CN18 1X4-3.5MM, CN19 1X4-3.5MM, CN2 1X4-3.5MM, CN20 1X4-3.5MM, CN21 1X4-3.5MM, CN22 1X4-3.5MM, CN23 1X4-3.5MM, CN24 1X4-3.5MM, CN25 1X4-3.5MM, CN26 1X4-3.5MM, CN27 1X4-3.5MM, CN28 1X4-3.5MM, CN29 1X4-3.5MM, CN3 1X4-3.5MM, CN30 1X4-3.5MM, CN31 1X4-3.5MM, CN32 1X4-3.5MM, CN33 1X4-3.5MM, CN34 1X4-3.5MM, CN4 1X4-3.5MM, CN5 1X4-3.5MM, CN6 1X4-3.5MM, CN7 1X4-3.5MM, CN8 1X4-3.5MM, CN9 1X4-3.5MM, Q1 16mhz, U2 MCP2551, U3 ARDUINO-MEGAFULL

Commit message: Ethernet connector-previous version
Parts:
- removed CN10, CN11, CN26, CN30, CN31, CN32, CN34, CN7, CN8, CN9: 1X4-3.5MM, Arduino_merg:1X04-3.5MM
- added ANALOG, ANALOG1, DIGITAL1, DIGITAL2, DIGITAL3, PWM: RJ45-8PTH, SparkFun-Connectors:RJ45-8
- moved CN13 0.65 mm to (89.0, 3.18)
Connections:
- net 2: now also PWM.1
- net 24: now also DIGITAL1.8
- net 25: now also DIGITAL1.7
- net 26: now also DIGITAL1.6
- net 27: now also DIGITAL1.5; no longer CN7.1
- net 28: now also DIGITAL1.4; no longer CN7.2
- net 29: now also DIGITAL1.3; no longer CN7.3
- net 3: now also PWM.2
- net 30: now also DIGITAL1.2; no longer CN7.4
- net 31: now also DIGITAL1.1; no longer CN8.1
- net 32: now also DIGITAL2.8; no longer CN8.2
- net 33: now also DIGITAL2.7; no longer CN8.3
- net 34: now also DIGITAL2.6; no longer CN8.4
- net 35: now also DIGITAL2.5; no longer CN9.1
- net 36: now also DIGITAL2.4; no longer CN9.2
- net 37: now also DIGITAL2.3; no longer CN9.3
- net 38: now also DIGITAL2.2; no longer CN9.4
- net 39: now also DIGITAL2.1; no longer CN10.1
- net 4: now also PWM.3
- net 40: now also DIGITAL3.8; no longer CN10.2
- net 41: now also DIGITAL3.7; no longer CN10.3
- net 42: now also DIGITAL3.6; no longer CN10.4
- net 43: now also DIGITAL3.5; no longer CN11.1
- net 44: now also DIGITAL3.4; no longer CN11.2
- net 45: now also DIGITAL3.3; no longer CN11.3
- net 46: now also DIGITAL3.2; no longer CN11.4
- net 47: now also DIGITAL3.1
- net 5: now also PWM.4
- net 6: now also PWM.5
- net 7: now also PWM.6
- net 8: now also PWM.7
- net 9: now also PWM.8
- net A0: now also ANALOG.1
- net A1: now also ANALOG.2
- net A10: now also ANALOG1.3
- net A11: now also ANALOG1.4
- net A12: now also ANALOG1.5
- net A13: now also ANALOG1.6
- net A14: now also ANALOG1.7
- net A15: now also ANALOG1.8
- net A2: now also ANALOG.3
- net A3: now also ANALOG.4
- net A4: now also ANALOG.5
- net A5: now also ANALOG.6
- net A6: now also ANALOG.7
- net A7: now also ANALOG.8
- net A8: now also ANALOG1.1
- net A9: now also ANALOG1.2
Routing:
- net VCC: track 253.8 -> 86.3 mm, vias 3 -> 0
- net GND: track 237.1 -> 114.0 mm
- net VCC1: track 57.6 -> 0.00 mm
- net 28: track 32.1 -> 0.00 mm
- net 46: track 26.6 -> 0.00 mm
- net 30: track 24.5 -> 0.00 mm
- net 27: track 24.2 -> 0.00 mm
- net 45: track 23.4 -> 0.00 mm
- net 44: track 22.1 -> 0.00 mm
- net 43: track 19.0 -> 0.00 mm
- net 42: track 17.7 -> 0.00 mm
- net 29: track 17.4 -> 0.00 mm
- net 41: track 14.5 -> 0.00 mm
- net 32: track 14.2 -> 0.00 mm
- net 40: track 13.6 -> 0.00 mm
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Other:
- board text removed: "27"
- board text removed: "28"
- board text removed: "29"
- board text removed: "30"
- board text removed: "31"
- board text removed: "32"
- board text removed: "33"
- board text removed: "34"
- board text removed: "35"
- board text removed: "36"
- board text removed: "37"
- board text removed: "38"
- board text removed: "39"
- board text removed: "40"
- board text removed: "41"
- board text removed: "42"
- board text removed: "43"
- board text removed: "44"
- board text removed: "45"
- board text removed: "46"

Commit message: Board with ethernet connectors.
Parts:
- removed CN33, CN6: 1X4-3.5MM, Arduino_merg:1X04-3.5MM
- moved ANALOG 57.1 mm to (97.0, 9.93)
- moved PWM 18.6 mm to (78.4, 76.3), turned to 180 degrees
- moved ANALOG1 15.4 mm to (96.1, 25.4)
- moved DIGITAL2 15.4 mm to (96.1, 56.3)
- moved DIGITAL3 15.4 mm to (96.1, 40.8)
- moved DIGITAL1 15.3 mm to (96.1, 71.8)
- moved CN13 0.33 mm to (89.0, 2.85)
Connections:
- removed net N$53: CN6.4
- net 24: no longer CN6.3
- net 25: no longer CN6.2
- net 26: no longer CN6.1
- net GND: now also U3.GND@4
Routing:
- net VCC: track 86.3 -> 276.1 mm
- net A0: track 28.4 -> 106.2 mm
- net A2: track 24.5 -> 96.3 mm
- net A1: track 25.4 -> 92.8 mm
- net 9: track 16.2 -> 82.4 mm
- net A3: track 23.5 -> 89.5 mm
- net A4: track 22.6 -> 88.0 mm
- net 8: track 15.2 -> 77.1 mm
- net A10: track 19.4 -> 79.3 mm
- net A6: track 20.7 -> 79.3 mm
- net 6: track 14.9 -> 70.6 mm
- net 7: track 15.8 -> 71.2 mm
- net A8: track 21.3 -> 75.8 mm
- net A7: track 19.7 -> 72.4 mm
- net A5: track 21.6 -> 70.7 mm
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
Commit message: Last version with correction.
Routing:
- net GND: track 114.2 -> 114.8 mm
Changed lines of the file:
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@@
 <description language="de">&lt;b&gt;EAGLE Design Rules&lt;/b&gt;
 &lt;p&gt;
-Die Standard-Design-Rules sind so gewählt, dass sie für
+Die Standard-Design-Rules sind so gewÃ¤hlt, dass sie fÃ¼r
 die meisten Anwendungen passen. Sollte ihre Platine
 besondere Anforderungen haben, treffen Sie die erforderlichen
@@
 <autorouter>
 <pass name="Default">
-<param name="RoutingGrid" value="50mil"/>
+<param name="RoutingGrid" value="6.25mil"/>
 <param name="AutoGrid" value="1"/>
 <param name="Efforts" value="1"/>
 <param name="TopRouterVariant" value="1"/>
 <param name="tpViaShape" value="round"/>
-<param name="PrefDir.1" value="a"/>
+<param name="PrefDir.1" value="*"/>
 <param name="PrefDir.2" value="0"/>
 <param name="PrefDir.3" value="0"/>
@@
 <param name="PrefDir.14" value="0"/>
 <param name="PrefDir.15" value="0"/>
-<param name="PrefDir.16" value="a"/>
+<param name="PrefDir.16" value="*"/>
 <param name="cfVia" value="8"/>
 <param name="cfNonPref" value="5"/>
@@
 <wire x1="14.6304" y1="30.9372" x2="14.526134375" y2="30.96958125" width="0.1524" layer="16"/>
 <wire x1="14.6304" y1="30.9372" x2="14.526115625" y2="30.9372" width="0.1524" layer="16"/>
-<wire x1="8.52" y1="25.4" x2="4.71" y2="25.4" width="0" layer="19" extent="16-16"/>
-<wire x1="14.526134375" y1="30.96958125" x2="8.52" y2="25.4" width="0" layer="19" extent="16-16"/>
-<wire x1="27.94" y1="15.24" x2="17.186240625" y2="13.952403125" width="0" layer="19" extent="16-16"/>
-<wire x1="83.82" y1="20.32" x2="87.294525" y2="2.85115625" width="0" layer="19" extent="1-1"/>
+<wire x1="90.805" y1="3.175" x2="90.794525" y2="2.85115625" width="0.1524" layer="1"/>
+<wire x1="90.805" y1="3.175" x2="90.747703125" y2="2.89795625" width="0.1524" layer="1"/>
 </signal>
 <signal name="VCC">
