File: arduino_nano_cbus_mux/eagle_mini.sch (EAGLE design)
At the start: 44 parts, among them J1 1X2-3.5MM, J2 1X2-3.5MM, M1 ARDUINO-PRO-MINI-5.0V

Commit message: update the last boards
Parts:
- removed JPD9, JPLG: (no value), SparkFun-Connectors:M03PTH
- JPLY: value (none) -> M02PTH; device SparkFun-Connectors:M03PTH -> SparkFun-Connectors:M02PTH
Connections:
- removed net JD9: JPD9.1
- removed net N$2: JPD9.3, R3.2, S2.3, S2.4
- removed net N$27: JPLG.2, R2.1
- net A0: no longer JPLG.3
- net A1: no longer JPLY.3
- net A5: now also R2.1
- net D1: no longer JPLG.1
- net D7: now also U$2.EN
- net D8: now also U$1.EN
- net D9: now also R3.2, S2.3, S2.4; no longer JPD9.2
- net GND: no longer U$1.EN, U$2.EN
