File: arduino_nano_cbus_mux/eagle_mini.brd (EAGLE design)
At the start: 90.5 x 71.4 mm, 44 parts, among them J1 1X2-3.5MM, J2 1X2-3.5MM, M1 ARDUINO-PRO-MINI-5.0V

Commit message: New layout for RFM69HC
Parts:
- removed JPD9, JPLG: (no value), SparkFun-Connectors:1X03
- JPLY: value (none) -> M02PTH; device SparkFun-Connectors:1X03 -> SparkFun-Connectors:1X02
- moved JPLY 51.1 mm to (-0.51, -4.06)
Connections:
- removed net JD9: JPD9.1
- removed net N$2: JPD9.3, R3.P$2, S2.3, S2.4
- removed net N$27: JPLG.2, R2.P$1
- net A0: no longer JPLG.3
- net A1: no longer JPLY.3
- net A5: now also R2.P$1
- net D1: no longer JPLG.1
- net D7: now also U$2.15
- net D8: now also U$1.15
- net D9: now also R3.P$2, S2.3, S2.4; no longer JPD9.2
- net GND: no longer U$1.15, U$2.15
Routing:
- net N$27: track 41.5 -> 0.00 mm
- net A5: track 103.5 -> 145.0 mm
- net N$2: track 23.7 -> 0.00 mm
- net D9: track 83.7 -> 107.1 mm
- net A1: track 145.9 -> 127.9 mm
