File: pb-led-matrix/pb-led-matrix.sch (EAGLE design)
At the start: 66 parts, among them X2 87758-2616

Commit message: update the last boards
Parts:
- removed X1: (no value), SparkFun-Connectors:DB25V
- removed X2: 87758-2616, con-molex:87758-2616
- added H1, H2, H3: MOUNT-HOLE3.6, holes:MOUNT-HOLE3.6
- added U1: 7826-0000PR, 3M_By_element14_Batch_1:7826-0000PR
- added X3: (no value), SparkFun-Connectors:F25VP
Connections:
- net N$26: now also U1.14; no longer X2-26.S
- net P1: now also U1.1, X3.1; no longer X1.1, X2-1.S
- net P10: now also U1.10, X3.10; no longer X1.10, X2-19.S
- net P11: now also U1.11, X3.11; no longer X1.11, X2-21.S
- net P12: now also U1.12, X3.12; no longer X1.12, X2-23.S
- net P13: now also U1.13, X3.13; no longer X1.13, X2-25.S
- net P14: now also U1.26, X3.14; no longer X1.14, X2-2.S
- net P15: now also U1.25, X3.15; no longer X1.15, X2-4.S
- net P16: now also U1.24, X3.16; no longer X1.16, X2-6.S
- net P17: now also U1.23, X3.17; no longer X1.17, X2-8.S
- net P18: now also U1.22, X3.18; no longer X1.18, X2-10.S
- net P19: now also U1.21, X3.19; no longer X1.19, X2-12.S
- net P2: now also U1.2, X3.2; no longer X1.2, X2-3.S
- net P20: now also U1.20, X3.20; no longer X1.20, X2-14.S
- net P21: now also U1.19, X3.21; no longer X1.21, X2-16.S
- net P22: now also U1.18, X3.22; no longer X1.22, X2-18.S
- net P23: now also U1.17, X3.23; no longer X1.23, X2-20.S
- net P24: now also U1.16, X3.24; no longer X1.24, X2-22.S
- net P25: now also U1.15, X3.25; no longer X1.25, X2-24.S
- net P3: now also U1.3, X3.3; no longer X1.3, X2-5.S
- net P4: now also U1.4, X3.4; no longer X1.4, X2-7.S
- net P5: now also U1.5, X3.5; no longer X1.5, X2-9.S
- net P6: now also U1.6, X3.6; no longer X1.6, X2-11.S
- net P7: now also U1.7, X3.7; no longer X1.7, X2-13.S
- net P8: now also U1.8, X3.8; no longer X1.8, X2-15.S
- net P9: now also U1.9, X3.9; no longer X1.9, X2-17.S
